File: ESP12E BOB_1.kicad_pcb (KiCad board)
At the start: 2 copper layers, 26.4 x 43.4 mm, 20 parts, among them M1 ESP-12E, P1 CONN_01X07, P2 CONN_01X13, P3 CONN_01X13, P4 CONN_01X01, P5 CONN_01X01, P6 CONN_01X01, P7 CONN_01X01, Q1 BSS138, Q2 BSS138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

Commit message: ESP12E board test review
Parts:
- added REF**: WireConnection_0-8mmDrill, Wire_Connections_Bridges:WireConnection_0-8mmDrill, F.Cu at (143.5, 63.5)
- added REF**: WireConnection_0-8mmDrill, Wire_Connections_Bridges:WireConnection_0-8mmDrill, F.Cu at (108.5, 63.5)
- added REF**: WireConnection_0-8mmDrill, Wire_Connections_Bridges:WireConnection_0-8mmDrill, F.Cu at (125.5, 87.9)
- added REF**: WireConnection_0-8mmDrill, Wire_Connections_Bridges:WireConnection_0-8mmDrill, F.Cu at (125.5, 37.3)
Other:
- board size 26.4 x 43.4 mm -> 39.1 x 54.9 mm
- board text added: "1. module 3.3V no connected. 2. UART connections 3. Keep board mounting holes 2mm. 4. Labels should be reflect on the baord."
